Commit message: 10/28 update

File: table_tennis_robot/pingpong_description/urdf/pingpong.gazebo.xacro (robot description, xacro)
@@ -5,12 +5,12 @@
       <dampingFactor>0.0</dampingFactor>
       <maxVel>100</maxVel>
-      <minDepth>0</minDepth>
-      <mu1>0.05</mu1>
-      <mu2>0.05</mu2>
+      <minDepth>0.001</minDepth>
+      <mu1>0.01</mu1>
+      <mu2>0.01</mu2>
       <fdir1>0 0 0</fdir1>
-      <kp>1e+5</kp>
-      <kd>1e-2</kd>
+      <!--<kp>1e+5</kp>-->
+      <kd>1.0</kd>
       <selfCollide>0</selfCollide>
-      <maxContacts>5</maxContacts>  <!-- set this to 1 and ball stops sliding with high angle -->
+      <maxContacts>10</maxContacts>  <!-- set this to 1 and ball stops sliding with high angle -->
       <!--<material>Gazebo/Orange</material>--> <!-- caution this overrwrites (dae) everything!!! -->
    </gazebo>

File: table_tennis_robot/table_description/urdf/tabletennis_table.gazebo.xacro (robot description, xacro)
@@ -5,14 +5,13 @@
          <gravity>1</gravity>
          <dampingFactor>0.0</dampingFactor>
-         <maxVel>1</maxVel>
-         <minDepth>0.0</minDepth>
+         <maxVel>1.0</maxVel>
+         <minDepth>1.0</minDepth>
          <mu1>0.5</mu1>
          <mu2>0.5</mu2>
          <fdir1>0 0 0</fdir1>
-         <kp>1e+10</kp>
-         <kd>1.0</kd>
-         <selfCollide>0</selfCollide>
-         <maxContacts>3</maxContacts>  <!-- set this to 1 and ball stops sliding with high angle -->
-         <material>Gazebo/Red</material> <!-- caution this overrwrites (dae) everything!!! -->
+         <kp>1e+7</kp>
+         <kd>1e-10</kd>
+         <selfCollide>1</selfCollide>
+         <maxContacts>10</maxContacts>  <!-- set this to 1 and ball stops sliding with high angle -->
       </gazebo>
    </xacro:macro>
