Commit message: modify URDF <mass> <inertia> tag, modify tabletennis table size, modeify robot name

File: table_tennis_robot/tabletennisrobot_description/urdf/TTbot.transmission.xacro (robot description, xacro)
@@ -7,8 +7,8 @@
             <type>transmission_interface/SimpleTransmission</type>
             <joint name="${prefix}joint_0">
-                <hardwareInterface>hardware_interface/PositionJointInterface</hardwareInterface>
+                <hardwareInterface>hardware_interface/VelocityJointInterface</hardwareInterface>
             </joint>
             <actuator name="${prefix}J0_motor">
-                <hardwareInterface>hardware_interface/PositionJointInterface</hardwareInterface>
+                <hardwareInterface>hardware_interface/VelocityJointInterface</hardwareInterface>
                 <mechanicalReduction>1</mechanicalReduction>
             </actuator>
@@ -17,8 +17,8 @@
             <type>transmission_interface/SimpleTransmission</type>
             <joint name="${prefix}joint_1">
-                <hardwareInterface>hardware_interface/PositionJointInterface</hardwareInterface>
+                <hardwareInterface>hardware_interface/VelocityJointInterface</hardwareInterface>
             </joint>
             <actuator name="${prefix}J1_motor">
-                <hardwareInterface>hardware_interface/PositionJointInterface</hardwareInterface>
+                <hardwareInterface>hardware_interface/VelocityJointInterface</hardwareInterface>
                 <mechanicalReduction>1</mechanicalReduction>
             </actuator>
@@ -27,8 +27,8 @@
             <type>transmission_interface/SimpleTransmission</type>
             <joint name="${prefix}joint_2">
-                <hardwareInterface>hardware_interface/PositionJointInterface</hardwareInterface>
+                <hardwareInterface>hardware_interface/VelocityJointInterface</hardwareInterface>
             </joint>
             <actuator name="${prefix}J2_motor">
-                <hardwareInterface>hardware_interface/PositionJointInterface</hardwareInterface>
+                <hardwareInterface>hardware_interface/VelocityJointInterface</hardwareInterface>
                 <mechanicalReduction>1</mechanicalReduction>
             </actuator>
@@ -37,8 +37,8 @@
             <type>transmission_interface/SimpleTransmission</type>
             <joint name="${prefix}joint_3">
-                <hardwareInterface>hardware_interface/PositionJointInterface</hardwareInterface>
+                <hardwareInterface>hardware_interface/VelocityJointInterface</hardwareInterface>
             </joint>
             <actuator name="${prefix}J3_motor">
-                <hardwareInterface>hardware_interface/PositionJointInterface</hardwareInterface>
+                <hardwareInterface>hardware_interface/VelocityJointInterface</hardwareInterface>
                 <mechanicalReduction>1</mechanicalReduction>
             </actuator>
@@ -47,8 +47,8 @@
             <type>transmission_interface/SimpleTransmission</type>
             <joint name="${prefix}joint_4">
-                <hardwareInterface>hardware_interface/PositionJointInterface</hardwareInterface>
+                <hardwareInterface>hardware_interface/VelocityJointInterface</hardwareInterface>
             </joint>
             <actuator name="${prefix}J4_motor">
-                <hardwareInterface>hardware_interface/PositionJointInterface</hardwareInterface>
+                <hardwareInterface>hardware_interface/VelocityJointInterface</hardwareInterface>
                 <mechanicalReduction>1</mechanicalReduction>
             </actuator>

File: table_tennis_robot/tabletennisrobot_description/urdf/TTbot.urdf.xacro (robot description, xacro)
@@ -12,6 +12,6 @@
 			<inertial>
 		    	<origin xyz="0 0 0" rpy="0 0 0" />
-       			<mass value="10" />
-       			<inertia ixx="0.0441803207364147" ixy="5.37433593375545E-07" ixz="0.004045564920652" iyy="0.0584309411563095" iyz="-4.8990117845347E-07" izz="0.0514875586171667" />
+       			<mass value="93.462" />
+       			<inertia ixx="13.838" ixy="0.0" ixz="0.0" iyy="95.310" iyz="0.0" izz="94.912" />
 		    </inertial>
       		<visual>
@@ -31,6 +31,6 @@
 			<inertial>
 		    	<origin xyz="0 0 0" rpy="0 0 0" />
-       			<mass value="10" />
-       			<inertia ixx="0.0441803207364147" ixy="5.37433593375545E-07" ixz="0.004045564920652" iyy="0.0584309411563095" iyz="-4.8990117845347E-07" izz="0.0514875586171667" />
+       			<mass value="4.462" />
+       			<inertia ixx="5.886E-02" ixy="0.0" ixz="0.0" iyy="1.426E-02" iyz="0.0" izz="6.193E-02" />
 		    </inertial>
       		<visual>
@@ -50,6 +50,6 @@
 			<inertial>
 		    	<origin xyz="${-0.125/2} 0 ${-0.125/2}" rpy="0 0 0" />
-       			<mass value="10" />
-       			<inertia ixx="0.0441803207364147" ixy="5.37433593375545E-07" ixz="0.004045564920652" iyy="0.0584309411563095" iyz="-4.8990117845347E-07" izz="0.0514875586171667" />
+       			<mass value="1.610" />
+       			<inertia ixx="9.545E-03" ixy="0.0" ixz="0.0" iyy="1.793E-03" iyz="0.0" izz="9.380E-03" />
 		    </inertial>
       		<visual>
@@ -69,6 +69,6 @@
 			<inertial>
 		    	<origin xyz="${-0.067/2} ${-0.015} ${-0.067/2}" rpy="0 0 0" />
-       			<mass value="10" />
-       			<inertia ixx="0.0441803207364147" ixy="5.37433593375545E-07" ixz="0.004045564920652" iyy="0.0584309411563095" iyz="-4.8990117845347E-07" izz="0.0514875586171667" />
+       			<mass value="9.078E-01" />
+       			<inertia ixx="9.568E-04" ixy="0.0" ixz="0.0" iyy="4.031E-02" iyz="0.0" izz="4.069E-02" />
 		    </inertial>
       		<visual>
@@ -88,6 +88,6 @@
 			<inertial>
 		    	<origin xyz="${-0.039/2} ${-0.023} ${-0.039/2}" rpy="0 0 0" />
-       			<mass value="10" />
-       			<inertia ixx="0.0441803207364147" ixy="5.37433593375545E-07" ixz="0.004045564920652" iyy="0.0584309411563095" iyz="-4.8990117845347E-07" izz="0.0514875586171667" />
+       			<mass value="3.270E-01" />
+       			<inertia ixx="1.203E-04" ixy="0.0" ixz="0.0" iyy="7.429E-3" iyz="0.0" izz="7.462E-3" />
 		    </inertial>
       		<visual>
@@ -107,6 +107,6 @@
 			<inertial>
 		    	<origin xyz="${-0.1+0.045/2} ${-0.01} ${-0.045/2}" rpy="0 ${0} 0" />
-       			<mass value="10" />
-       			<inertia ixx="0.0441803207364147" ixy="5.37433593375545E-07" ixz="0.004045564920652" iyy="0.0584309411563095" iyz="-4.8990117845347E-07" izz="0.0514875586171667" />
+       			<mass value="1.331E-01" />
+       			<inertia ixx="3.713E-05" ixy="0.0" ixz="0.0" iyy="2.703E-04" iyz="0.0" izz="2.622E-04" />
 		    </inertial>
       		<visual>
