Commit message: add joint6 to TTbot

File: table_tennis_robot/tabletennisrobot_description/urdf/TTbot.gazebo.xacro (robot description, xacro)
@@ -60,4 +60,10 @@
                 <material>Gazebo/Grey</material>
             </gazebo>
+            <gazebo reference="joint_5_link">
+                <mu1>1</mu1>
+                <mu2>1</mu2>
+                <selfCollide>true</selfCollide>
+                <material>Gazebo/Red</material>
+            </gazebo>
         </xacro:if>
     </xacro:macro>

File: table_tennis_robot/tabletennisrobot_description/urdf/TTbot.transmission.xacro (robot description, xacro)
@@ -54,4 +54,14 @@
             </actuator>
         </transmission>
+        <transmission name="${prefix}J5_trans">
+            <type>transmission_interface/SimpleTransmission</type>
+            <joint name="${prefix}joint_5">
+                <hardwareInterface>hardware_interface/VelocityJointInterface</hardwareInterface>
+            </joint>
+            <actuator name="${prefix}J5_motor">
+                <hardwareInterface>hardware_interface/VelocityJointInterface</hardwareInterface>
+                <mechanicalReduction>1</mechanicalReduction>
+            </actuator>
+        </transmission>
     </xacro:macro>
 </robot>

File: table_tennis_robot/tabletennisrobot_description/urdf/TTbot.urdf.xacro (robot description, xacro)
@@ -113,5 +113,5 @@
 		        <origin xyz="${-0.1+0.045/2} ${-0.01} ${-0.045/2}" rpy="0 ${0} 0" />
         		<geometry>
-        			<mesh filename="package://tabletennisrobot_description/meshes/visual/joint_4_link.dae" />
+        			<mesh filename="package://tabletennisrobot_description/meshes/visual/joint_4_link_DLC.dae" />
 		        </geometry>
 		    </visual>
@@ -119,24 +119,24 @@
         		<origin xyz="${-0.1+0.045/2} ${-0.01} ${-0.045/2}" rpy="0 ${0} 0" />
         		<geometry>
-          			<mesh filename="package://tabletennisrobot_description/meshes/visual/joint_4_link.dae" />
+          			<mesh filename="package://tabletennisrobot_description/meshes/visual/joint_4_link_DLC.dae" />
 		        </geometry>
  		    </collision>
     	</link>
-		<link name="${prefix}racket_link" >
+		<link name="${prefix}joint_5_link" >
 			<inertial>
-		    	<origin xyz="${0} ${0} ${0}" rpy="0 ${0} ${-pi/6}" />
+		    	<origin xyz="${-0.0225} ${0} ${-0.015}" rpy="0 ${0} ${0}" />
        			<mass value="8.5E-02" />
        			<inertia ixx="3.713E-05" ixy="0.0" ixz="0.0" iyy="2.703E-04" iyz="0.0" izz="2.622E-04" />
 		    </inertial>
       		<visual>
-		        <origin xyz="${0} ${0} ${0}" rpy="0 ${0} ${-pi/6}" />
+		        <origin xyz="${-0.0225} ${0} ${-0.015}" rpy="0 ${0} ${0}" />
         		<geometry>
-        			<mesh filename="package://tabletennisrobot_description/meshes/visual/racket3_1.dae" />
+        			<mesh filename="package://tabletennisrobot_description/meshes/visual/joint_5_link_DLC.dae" />
 		        </geometry>
 		    </visual>
       		<collision>
-				<origin xyz="${0} ${0} ${0}" rpy="0 ${0} ${-pi/6}" />
+				<origin xyz="${-0.0225} ${0} ${-0.015}" rpy="0 ${0} ${0}" />
         		<geometry>
-          			<mesh filename="package://tabletennisrobot_description/meshes/visual/racket3_1.dae" />
+          			<mesh filename="package://tabletennisrobot_description/meshes/visual/joint_5_link_DLC.dae" />
 		        </geometry>
  		    </collision>
@@ -183,8 +183,11 @@
         	<axis xyz="0 1 0"/>
     	</joint>
-		<joint name="${prefix}joint_racket" type="fixed">
+		<joint name="${prefix}joint_5" type="revolute">
 			<parent link="${prefix}joint_4_link"/>
-        	<child link="${prefix}racket_link"/>
-			<origin xyz="${-0.26-0.0325} ${0.015} ${0}" rpy="0 ${pi/2} ${0}" />
+        	<child link="${prefix}joint_5_link"/>
+			<origin xyz="${-0.0765} ${0.0435} ${0.001}" rpy="0 ${0} ${pi/2}" />
+			<limit effort="1000.0" lower="${-pi}" upper="${pi}" velocity="1.0"/>
+        	<dynamics damping="0.0" friction="0.0"/>
+			<axis xyz="0 1 0"/>
     	</joint>
 		<!-- gazebo and transmission -->
