Commit message: update 12/10

File: table_tennis_robot/tabletennisrobot_description/urdf/TTbot.urdf.xacro (robot description, xacro)
@@ -123,4 +123,23 @@
  		    </collision>
     	</link>
+		<link name="${prefix}racket_link" >
+			<inertial>
+		    	<origin xyz="${0} ${0} ${0}" rpy="0 ${0} ${-pi/6}" />
+       			<mass value="8.5E-02" />
+       			<inertia ixx="3.713E-05" ixy="0.0" ixz="0.0" iyy="2.703E-04" iyz="0.0" izz="2.622E-04" />
+		    </inertial>
+      		<visual>
+		        <origin xyz="${0} ${0} ${0}" rpy="0 ${0} ${-pi/6}" />
+        		<geometry>
+        			<mesh filename="package://tabletennisrobot_description/meshes/visual/racket3_1.dae" />
+		        </geometry>
+		    </visual>
+      		<collision>
+				<origin xyz="${0} ${0} ${0}" rpy="0 ${0} ${-pi/6}" />
+        		<geometry>
+          			<mesh filename="package://tabletennisrobot_description/meshes/visual/racket3_1.dae" />
+		        </geometry>
+ 		    </collision>
+    	</link>
     	<!-- joints: -->
 		<joint name="${prefix}joint_0" type="prismatic">
@@ -164,4 +183,9 @@
         	<axis xyz="0 1 0"/>
     	</joint>
+		<joint name="${prefix}joint_racket" type="fixed">
+			<parent link="${prefix}joint_4_link"/>
+        	<child link="${prefix}racket_link"/>
+			<origin xyz="${-0.26-0.0325} ${0.015} ${0}" rpy="0 ${pi/2} ${0}" />
+    	</joint>
 		<!-- gazebo and transmission -->
 		<xacro:TTbot_transmission prefix="${prefix}" />

Commit message: can pub 5 joint pos and vel (real motor)

File: table_tennis_robot/tabletennisrobot_description/urdf/TTbot.urdf.xacro (robot description, xacro)
@@ -148,5 +148,5 @@
     		<child link = "${prefix}slide_link" />
     		<axis xyz="1 0 0" />
-    		<limit effort="150" lower="0.2" upper="1.25" velocity="0.5" />
+    		<limit effort="150" lower="0.2" upper="1.25" velocity="1.0" />
     		<dynamics damping="0.0" friction="0.0"/>
   		</joint>
@@ -155,5 +155,5 @@
         	<child link="${prefix}joint_1_link"/>
 			<origin xyz="${0.147/2} ${0.225} ${0.15/2}" rpy="0 0 0" />
-        	<limit effort="1000.0" lower="${-pi*3/4}" upper="${pi*3/4}" velocity="0.5"/>
+        	<limit effort="1000.0" lower="${-pi*3/4}" upper="${pi*3/4}" velocity="10.0"/>
         	<dynamics damping="0.0" friction="0.0"/>
         	<axis xyz="0 1 0"/>
@@ -163,5 +163,5 @@
         	<child link="${prefix}joint_2_link"/>
 			<origin xyz="${0.05} ${0.091} ${0}" rpy="0 0 ${pi/2}" />
-        	<limit effort="1000.0" lower="${-pi*3/4}" upper="${pi*3/4}" velocity="0.5"/>
+        	<limit effort="1000.0" lower="${-pi*3/4}" upper="${pi*3/4}" velocity="1.0"/>
         	<dynamics damping="0.0" friction="0.0"/>
         	<axis xyz="0 1 0"/>
@@ -171,5 +171,5 @@
         	<child link="${prefix}joint_3_link"/>
 			<origin xyz="${0.253} ${0.082-0.015} ${0}" rpy="${pi} 0 0" />
-        	<limit effort="1000.0" lower="${-pi*3/4}" upper="${pi*3/4}" velocity="0.5"/>
+        	<limit effort="1000.0" lower="${-pi*3/4}" upper="${pi*3/4}" velocity="1.0"/>
         	<dynamics damping="0.0" friction="0.0"/>
         	<axis xyz="0 1 0"/>
@@ -179,5 +179,5 @@
         	<child link="${prefix}joint_4_link"/>
 			<origin xyz="${0.216} ${0.04-0.023} ${0}" rpy="0 0 ${pi}" />
-        	<limit effort="1000.0" lower="${-pi*3/4}" upper="${pi*3/4}" velocity="0.5"/>
+        	<limit effort="1000.0" lower="${-pi*3/4}" upper="${pi*3/4}" velocity="1.0"/>
         	<dynamics damping="0.0" friction="0.0"/>
         	<axis xyz="0 1 0"/>

Commit message: sync ral and sim, TTbot joint1 change

File: table_tennis_robot/tabletennisrobot_description/urdf/TTbot.urdf.xacro (robot description, xacro)
@@ -154,6 +154,6 @@
 			<parent link="${prefix}slide_link"/>
         	<child link="${prefix}joint_1_link"/>
-			<origin xyz="${0.147/2} ${0.225} ${0.15/2}" rpy="0 0 0" />
-        	<limit effort="1000.0" lower="${-pi*3/4}" upper="${pi*3/4}" velocity="10.0"/>
+			<origin xyz="${0.147/2} ${0.225} ${0.15/2}" rpy="0 ${pi} ${0}" />
+        	<limit effort="1000.0" lower="${-pi}" upper="${pi}" velocity="10.0"/>
         	<dynamics damping="0.0" friction="0.0"/>
         	<axis xyz="0 1 0"/>
@@ -163,5 +163,5 @@
         	<child link="${prefix}joint_2_link"/>
 			<origin xyz="${0.05} ${0.091} ${0}" rpy="0 0 ${pi/2}" />
-        	<limit effort="1000.0" lower="${-pi*3/4}" upper="${pi*3/4}" velocity="1.0"/>
+        	<limit effort="1000.0" lower="${-pi}" upper="${pi}" velocity="1.0"/>
         	<dynamics damping="0.0" friction="0.0"/>
         	<axis xyz="0 1 0"/>
@@ -171,5 +171,5 @@
         	<child link="${prefix}joint_3_link"/>
 			<origin xyz="${0.253} ${0.082-0.015} ${0}" rpy="${pi} 0 0" />
-        	<limit effort="1000.0" lower="${-pi*3/4}" upper="${pi*3/4}" velocity="1.0"/>
+        	<limit effort="1000.0" lower="${-pi}" upper="${pi}" velocity="1.0"/>
         	<dynamics damping="0.0" friction="0.0"/>
         	<axis xyz="0 1 0"/>
@@ -179,5 +179,5 @@
         	<child link="${prefix}joint_4_link"/>
 			<origin xyz="${0.216} ${0.04-0.023} ${0}" rpy="0 0 ${pi}" />
-        	<limit effort="1000.0" lower="${-pi*3/4}" upper="${pi*3/4}" velocity="1.0"/>
+        	<limit effort="1000.0" lower="${-pi}" upper="${pi}" velocity="1.0"/>
         	<dynamics damping="0.0" friction="0.0"/>
         	<axis xyz="0 1 0"/>

Commit message: pub robot_status to rviz,unified cmd can pub6joint

File: table_tennis_robot/tabletennisrobot_description/urdf/TTbot.urdf.xacro (robot description, xacro)
@@ -186,5 +186,5 @@
 			<parent link="${prefix}joint_4_link"/>
         	<child link="${prefix}joint_5_link"/>
-			<origin xyz="${-0.0765} ${0.0435} ${0.001}" rpy="0 ${0} ${pi/2}" />
+			<origin xyz="${-0.0765} ${0.0435} ${0.001}" rpy="0 ${pi/2} ${pi/2}" />
 			<limit effort="1000.0" lower="${-pi}" upper="${pi}" velocity="1.0"/>
         	<dynamics damping="0.0" friction="0.0"/>

Commit message: update 3/17

File: table_tennis_robot/tabletennisrobot_description/urdf/TTbot.urdf.xacro (robot description, xacro)
@@ -144,9 +144,10 @@
     	<!-- joints: -->
 		<joint name="${prefix}joint_0" type="prismatic">
-    		<origin xyz="0.0 0.4 0.621" rpy="${pi/2} 0 0" />
+    		<origin xyz="0.7265 0.4 0.621" rpy="${pi/2} 0 0" />
     		<parent link="${prefix}base_link" />
     		<child link = "${prefix}slide_link" />
     		<axis xyz="1 0 0" />
-    		<limit effort="150" lower="0.2" upper="1.25" velocity="1.0" />
+    		<limit effort="150" lower="-0.5" upper="0.5" velocity="1.0" />
+<!--    		<limit effort="150" lower="0.2" upper="1.25" velocity="1.0" />-->
     		<dynamics damping="0.0" friction="0.0"/>
   		</joint>
