Commit message: modify table, ball, link5 param(maxVel)

File: table_tennis_robot/table_description/urdf/tabletennis_table.gazebo.xacro (robot description, xacro)
@@ -5,8 +5,8 @@
          <gravity>1</gravity>
          <dampingFactor>0.0</dampingFactor>
-         <maxVel>1.0</maxVel>
-         <minDepth>1.0</minDepth>
-         <mu1>0.5</mu1>
-         <mu2>0.5</mu2>
+         <maxVel>100.0</maxVel>
+         <minDepth>0.0</minDepth>
+         <mu1>5.0</mu1>
+         <mu2>5.0</mu2>
          <fdir1>0 0 0</fdir1>
          <kp>1e+7</kp>
@@ -14,4 +14,12 @@
          <selfCollide>1</selfCollide>
          <maxContacts>10</maxContacts>  <!-- set this to 1 and ball stops sliding with high angle -->
+         <collision>
+            <surface>
+               <bounce>
+                  <restitution_coefficient>1.0</restitution_coefficient>
+                  <threshold>0.0</threshold>
+               </bounce>
+            </surface>
+         </collision>
       </gazebo>
    </xacro:macro>

File: table_tennis_robot/table_description/urdf/tabletennis_table.urdf.xacro (robot description, xacro)
@@ -2,5 +2,5 @@
 <robot xmlns:controller="http://playerstage.sourceforge.net/gazebo/xmlschema/#controller" xmlns:interface="http://ros.org/wiki/xacro" xmlns:sensor="http://playerstage.sourceforge.net/gazebo/xmlschema/#sensor" xmlns:xacro="http://ros.org/wiki/xacro" name="$(arg tabletennis_table_name)">
    <xacro:include filename="$(find table_description)/urdf/tabletennis_table.gazebo.xacro" />
-   <xacro:property name="scale_size" value="0.5" />
+   <xacro:property name="scale_size" value="1.0" />
    <xacro:macro name="tabletennis_table_macro" params="prefix">
       <material name="blue">
@@ -11,5 +11,5 @@
          <origin rpy="0 0 0" xyz="0 0 0" />
          <geometry>
-            <mesh filename="package://table_description/models/tabletennis_table/meshes/tabletennis_table.dae" scale="${scale_size*1} ${scale_size*1} ${scale_size*1}" />
+            <mesh filename="package://table_description/models/tabletennis_table/meshes/tabletennis_table_realsize.dae" scale="${scale_size*1} ${scale_size*1} ${scale_size*1}" />
          </geometry>
          <cast_shadows>1</cast_shadows>
@@ -26,5 +26,5 @@
             <origin rpy="0 0 0" xyz="0 0 0" />
             <geometry>
-               <mesh filename="package://table_description/models/tabletennis_table/meshes/tabletennis_table.dae" scale="${scale_size*1} ${scale_size*1} ${scale_size*1}" />
+               <mesh filename="package://table_description/models/tabletennis_table/meshes/tabletennis_table_realsize.dae" scale="${scale_size*1} ${scale_size*1} ${scale_size*1}" />
             </geometry>
          </collision>

File: table_tennis_robot/tabletennisrobot_description/urdf/TTbot.gazebo.xacro (robot description, xacro)
@@ -29,4 +29,12 @@
                 <selfCollide>true</selfCollide>
                 <material>Gazebo/DarkGrey</material>
+                <collision>
+                    <surface>
+                        <bounce>
+                            <restitution_coefficient>1.0</restitution_coefficient>
+                            <threshold>0.0</threshold>
+                        </bounce>
+                    </surface>
+                </collision>
             </gazebo>
             <gazebo reference="slide_link">
@@ -61,8 +69,19 @@
             </gazebo>
             <gazebo reference="joint_5_link">
-                <mu1>1</mu1>
-                <mu2>1</mu2>
+                <mu1>5</mu1>
+                <mu2>5</mu2>
+                <kp>10000000.0</kp>
+                <minDepth>0.001</minDepth>
+                <maxVel>10</maxVel>
                 <selfCollide>true</selfCollide>
                 <material>Gazebo/Red</material>
+                <collision>
+                    <surface>
+                        <bounce>
+                            <restitution_coefficient>1.0</restitution_coefficient>
+                            <threshold>0.0</threshold>
+                        </bounce>
+                    </surface>
+                </collision>
             </gazebo>
         </xacro:if>
